File: gizmo.kicad_pcb (KiCad board)
At the start: 2 copper layers, 119.4 x 96.5 mm, 143 parts, among them J1 Power In, J10 GPIO 11, J11 GPIO 12, J12 Servo GPIO 21, J13 Servo GPIO 20, J14 Servo GPIO 19, J15 Servo GPIO 18, J2 System Breakout, J20 ADC 2, J21 ADC 1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

Commit message: Problem: Silkscreen too large
Solution: Shrink it
Other:
- board text added: "v1.1"
- board text removed: "v01.01.r1"
